File: hw/ADC_Test.kicad_pcb (KiCad board)
At the start: 2 copper layers, 125 x 21.5 mm, 105 parts, among them J1 SMA SENSOR IN, J3 PMOD (ZedBoard), J4 SMA MON, J7 3V3 IN, U1 OPA2365, U2 OPA2365, U3 THS4531, U4 ADS7057, U6 TLV7022, U9 TLV7022

Commit message: Listener filter fix found by the netlist simulation: R36 10k, C41 22 pF, R39/R40 15k; sim/netlist_verify.py; manual and README updated
Co-Authored-By: Claude Sonnet 5.5 <noreply@anthropic.com>
Parts:
- C41: value 100pF C0G -> 22pF C0G
- R36: value 2.2k -> 10k
- R39, R40: value 18k -> 15k

Commit message: Power: 5-pin SMU header J7 replaces JP2/JP4/JP5/JP6 and the 2-pin header; top silkscreen with TP and IC numbers; slides and README updated
Co-Authored-By: Claude Sonnet 5.5 <noreply@anthropic.com>
Parts:
- removed JP2: LISTENER LINK, Jumper:SolderJumper-2_P1.3mm_Bridged_Pad1.0x1.5mm
- removed JP4: AVDD LINK, Jumper:SolderJumper-2_P1.3mm_Bridged_Pad1.0x1.5mm
- removed JP5: DVDD LINK, Jumper:SolderJumper-2_P1.3mm_Bridged_Pad1.0x1.5mm
- removed JP6: PMOD 3V3, Jumper:SolderJumper-2_P1.3mm_Bridged_Pad1.0x1.5mm
- J7: value 3V3 IN -> POWER / SMU; footprint Connector_PinHeader_2.54mm:PinHeader_1x02_P2.54mm_Vertical -> Connector_PinHeader_2.54mm:PinHeader_1x05_P2.54mm_Vertical
- moved TP11 7.03 mm to (204.6, 110.6)
- moved J7 2.62 mm to (198.0, 106.6), turned to 90 degrees
- moved C9 0.57 mm to (194.6, 106.9)
Connections:
- C19 pad 1: DVDD -> +3V3
- C20 pad 1: DVDD -> +3V3
- C28 pad 1: +3V3_L -> +3V3
- C45 pad 1: +3V3_L -> +3V3
- J7 pad 1: +3V3 -> +3V3_PMOD
- J7 pad 2: GND -> +3V3
- R21 pad 1: +3V3_L -> +3V3
- R34 pad 1: AVDD_IN -> +3V3_C
- U4 pad 4: DVDD -> +3V3
- U6 pad 8: +3V3_L -> +3V3
- U9 pad 8: +3V3_L -> +3V3
Routing:
- net +3V3_L: track 120.2 -> 0.00 mm, vias 5 -> 0
- net DVDD: track 42.5 -> 0.00 mm, vias 3 -> 0
- net +3V3_PMOD: track 14.8 -> 28.7 mm, vias 1 -> 0
- net VOCM: track 67.8 -> 54.0 mm
- net VMID5: track 97.2 -> 85.5 mm
- net SIG_IN: track 53.5 -> 41.9 mm
- net MON: track 89.6 -> 78.1 mm
- net +3V3: track 151.1 -> 161.5 mm, vias 7 -> 9
- net AINP: track 28.1 -> 37.4 mm, vias 0 -> 3
- net AVDD: track 53.0 -> 44.0 mm, vias 3 -> 4
- net GN_FB: track 10.5 -> 18.8 mm
- net +3V3_C: track 143.0 -> 135.4 mm
- net TH2M: track 31.3 -> 38.8 mm, vias 0 -> 3
- net BIG_N: track 131.1 -> 137.4 mm, vias 1 -> 3
- net GAIN_OUT: track 38.5 -> 43.9 mm, vias 0 -> 2
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Other:
- board text added: "TP10"
- board text added: "TP11"
- board text added: "TP12"
- board text added: "TP13"
- board text added: "TP14"
- board text added: "TP15"
- board text added: "TP16"
- board text added: "TP17"
- board text added: "TP18"
- board text added: "TP19"
- board text added: "TP20"
- board text added: "TP3"
- board text added: "TP4"
- board text added: "TP5"
- board text added: "TP6"
- board text added: "TP7"
- board text added: "TP8"
- board text added: "TP9"
- board text added: "U1"
- board text added: "U2"
- board text added: "U3"
- board text added: "U4"
- board text added: "U6"
- board text added: "U9"
- board text removed: "DVDD"
- board text removed: "LISTEN"
- board text removed: "PMOD 3V3"
