File: hw/ADC_Test.kicad_pcb (KiCad board)
At the start: 2 copper layers, 125 x 21.5 mm, 101 parts, among them J1 SMA SENSOR IN, J3 PMOD (ZedBoard), J4 SMA MON, J7 POWER / SMU, U1 OPA2365, U2 OPA2365, U3 THS4531, U4 ADS7057, U6 TLV7022, U9 TLV7022

Commit message: Silk: TP and JP labels centred on their pads, J7 pin legend, tidy back panel (AFE Test Board with logo, TP table, PMOD and J7 legends)
Co-Authored-By: Claude Sonnet 5.5 <noreply@anthropic.com>
Other:
- board text added: "1"
- board text added: "2"
- board text added: "3"
- board text added: "3 SENSE+ 4 SENSE- 5 FORCE-"
- board text added: "4"
- board text added: "5"
- board text added: "ADS7057 v3 Auselia 2026-10"
- board text added: "AFE Test Board"
- board text added: "F+"
- board text added: "F-"
- board text added: "J7 1 ONBOARD+ 2 FORCE+"
- board text added: "JP1"
- board text added: "JP1 head power"
- board text added: "JP3"
- board text added: "JP3 capture rail"
- board text added: "ON+"
- board text added: "S+"
- board text added: "S-"
- board text added: "TP10 AIN-"
- board text added: "TP11 3V3"
- board text added: "TP12 AVDD"
- board text added: "TP13 VMID5"
- board text added: "TP14 VOCM"
- board text added: "TP15 LST"
- board text added: "TP16 WAKE_N"
- board text added: "TP17 BIG_N"
- board text added: "TP18 REFL"
- board text added: "TP19 GND"
- board text added: "TP20 GND"
- board text added: "TP3 SIG_IN"
- board text added: "TP4 HPF"
- board text added: "TP5 GAIN"
- board text added: "TP6 LPF"
- board text added: "TP7 DRV+"
- board text added: "TP8 DRV-"
- board text added: "TP9 AIN+"
- board text removed: "3V3"
- board text removed: "ADS7057 test board v3"
- board text removed: "AIN+"
- board text removed: "AIN-"
- board text removed: "AVDD"
- board text removed: "Auselia 2026-10"
- board text removed: "BIG"
- board text removed: "CAPTURE"
- board text removed: "DRV+"
- board text removed: "DRV-"
- board text removed: "GAIN"
- board text removed: "GND"
- board text removed: "HEAD"
- board text removed: "HPF"
- board text removed: "LPF"
- board text removed: "LST"
- board text removed: "MID5"
- board text removed: "REFL"
- board text removed: "SIG"
- board text removed: "VOCM"
- board text removed: "WAKE"

Commit message: Head: +/- silk, U8 CPL rotation 0; main board silk says v1
Co-Authored-By: Claude Sonnet 5.5 <noreply@anthropic.com>
Other:
- board text added: "ADS7057 v1 Auselia 2026-10"
- board text removed: "ADS7057 v3 Auselia 2026-10"
Changed lines of the file:
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@@
 		)
 	)
-	(gr_text "ADS7057 v3   Auselia 2026-10"
+	(gr_text "ADS7057 v1   Auselia 2026-10"
 		(at 158 118.8 0)
 		(layer "B.SilkS")

Commit message: Back silkscreen spread out; Auselia / AFE Test Board v1 title
Co-Authored-By: Claude Sonnet 5.5 <noreply@anthropic.com>
Other:
- board text added: "AFE Test Board v1 2026-10"
- board text added: "Auselia"
- board text removed: "ADS7057 v1 Auselia 2026-10"
- board text removed: "AFE Test Board"
Changed lines of the file:
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@@
 	(gr_poly
 		(pts
-			(xy 161.7 118.449999) (xy 161.714978 118.221975) (xy 161.7586 118.009475) (xy 161.828899 117.812718)
-			(xy 161.923906 117.631924) (xy 162.041654 117.46731) (xy 162.180174 117.319096) (xy 162.3375 117.1875)
-			(xy 162.511661 117.07274) (xy 162.700692 116.975036) (xy 162.902623 116.894606) (xy 163.115488 116.831669)
-			(xy 163.337317 116.786443) (xy 163.566144 116.759147) (xy 163.8 116.75) (xy 163.785021 116.980867)
-			(xy 163.741399 117.20102) (xy 163.6711 117.408928) (xy 163.576093 117.603061) (xy 163.458345 117.781887)
-			(xy 163.319825 117.943877) (xy 163.1625 118.087499) (xy 162.988338 118.211224) (xy 162.799307 118.31352)
-			(xy 162.597376 118.392857) (xy 162.384511 118.447704) (xy 162.162682 118.47653) (xy 161.933855 118.477806)
+			(xy 139.799999 118.649999) (xy 139.814978 118.421975) (xy 139.8586 118.209475) (xy 139.928899 118.012718)
+			(xy 140.023906 117.831924) (xy 140.141654 117.66731) (xy 140.280174 117.519096) (xy 140.4375 117.3875)
+			(xy 140.611661 117.27274) (xy 140.800692 117.175036) (xy 141.002623 117.094606) (xy 141.215488 117.031669)
+			(xy 141.437317 116.986443) (xy 141.666144 116.959147) (xy 141.9 116.95) (xy 141.885021 117.180867)
+			(xy 141.841399 117.40102) (xy 141.7711 117.608928) (xy 141.676093 117.803061) (xy 141.558345 117.981887)
+			(xy 141.419825 118.143877) (xy 141.2625 118.2875) (xy 141.088338 118.411224) (xy 140.899307 118.51352)
+			(xy 140.697376 118.592857) (xy 140.484511 118.647704) (xy 140.262682 118.67653) (xy 140.033855 118.677806)
 		)
 		(stroke
@@
 	)
 	(gr_arc
-		(start 159.896558 117.309999)
-		(mid 159.5 116.049999)
-		(end 159.896558 114.789999)
+		(start 137.996558 117.509999)
+		(mid 137.6 116.25)
+		(end 137.996558 114.99)
 		(stroke
 			(width 0.36)
@@
 	)
 	(gr_arc
-		(start 160.551087 116.85)
-		(mid 160.3 116.05)
-		(end 160.551087 115.25)
+		(start 138.651087 117.05)
+		(mid 138.4 116.25)
+		(end 138.651087 115.45)
 		(stroke
 			(width 0.36)
@@
 	)
 	(gr_circle
-		(center 161.7 116.05)
-		(end 161.1 116.05)
+		(center 139.799999 116.25)
+		(end 139.2 116.25)
 		(stroke
 			(width 0.05)
@@
 	)
 	(gr_line
-		(start 161.7 119.449999)
-		(end 161.7 114.85)
+		(start 139.799999 119.649999)
+		(end 139.799999 115.05)
 		(stroke
 			(width 0.5)
@@
 		)
 	)
-	(gr_text "ADS7057 v1   Auselia 2026-10"
-		(at 158 118.8 0)
-		(layer "B.SilkS")
-		(effects
-			(font
-				(size 0.8 0.8)
-				(thickness 0.15)
-			)
-			(justify left mirror)
-		)
-	)
 	(gr_text "TP15 LST"
-		(at 166 103.4 0)
+		(at 158 103.4 0)
 		(layer "B.SilkS")
 		(effects
@@
 	)
 	(gr_text "TP16 WAKE_N"
-		(at 166 104.65 0)
+		(at 158 104.65 0)
 		(layer "B.SilkS")
 		(effects
@@
 	)
 	(gr_text "TP17 BIG_N"
-		(at 166 105.9 0)
+		(at 158 105.9 0)
 		(layer "B.SilkS")
 		(effects
@@
 	)
 	(gr_text "TP18 REFL"
-		(at 166 107.15 0)
+		(at 158 107.15 0)
 		(layer "B.SilkS")
 		(effects
@@
 	)
 	(gr_text "TP19 GND"
-		(at 166 108.4 0)
+		(at 158 108.4 0)
 		(layer "B.SilkS")
 		(effects
@@
 	)
 	(gr_text "TP20 GND"
-		(at 166 109.65 0)
+		(at 158 109.65 0)
 		(layer "B.SilkS")
 		(effects
@@
 	)
 	(gr_text "J7 1 ONBOARD+ 2 FORCE+"
-		(at 166 111.9 0)
+		(at 164 112.2 0)
 		(layer "B.SilkS")
 		(effects
@@
 	)
 	(gr_text "3 SENSE+ 4 SENSE- 5 FORCE-"
-		(at 166 113.2 0)
+		(at 164 113.6 0)
 		(layer "B.SilkS")
 		(effects
@@
 	)
 	(gr_text "TP9 AIN+"
-		(at 176 103.4 0)
+		(at 173 103.4 0)
 		(layer "B.SilkS")
 		(effects
@@
 	)
 	(gr_text "TP10 AIN-"
-		(at 176 104.65 0)
+		(at 173 104.65 0)
 		(layer "B.SilkS")
 		(effects
@@
 	)
 	(gr_text "TP11 3V3"
-		(at 176 105.9 0)
+		(at 173 105.9 0)
 		(layer "B.SilkS")
 		(effects
@@
 	)
 	(gr_text "TP12 AVDD"
-		(at 176 107.15 0)
+		(at 173 107.15 0)
 		(layer "B.SilkS")
 		(effects
@@
 	)
 	(gr_text "TP13 VMID5"
-		(at 176 108.4 0)
+		(at 173 108.4 0)
 		(layer "B.SilkS")
 		(effects
@@
 	)
 	(gr_text "TP14 VOCM"
-		(at 176 109.65 0)
+		(at 173 109.65 0)
 		(layer "B.SilkS")
 		(effects
@@
 	)
 	(gr_text "TP3 SIG_IN"
-		(at 186 103.4 0)
+		(at 188 103.4 0)
 		(layer "B.SilkS")
 		(effects
@@
 	)
 	(gr_text "TP4 HPF"
-		(at 186 104.65 0)
+		(at 188 104.65 0)
 		(layer "B.SilkS")
 		(effects
@@
 	)
 	(gr_text "TP5 GAIN"
-		(at 186 105.9 0)
+		(at 188 105.9 0)
 		(layer "B.SilkS")
 		(effects
@@
 	)
 	(gr_text "TP6 LPF"
-		(at 186 107.15 0)
+		(at 188 107.15 0)
 		(layer "B.SilkS")
 		(effects
@@
 	)
 	(gr_text "TP7 DRV+"
-		(at 186 108.4 0)
+		(at 188 108.4 0)
 		(layer "B.SilkS")
 		(effects
@@
 	)
 	(gr_text "TP8 DRV-"
-		(at 186 109.65 0)
+		(at 188 109.65 0)
 		(layer "B.SilkS")
 		(effects
@@
 	)
 	(gr_text "JP1 head power"
-		(at 186 111.9 0)
+		(at 188 112.2 0)
 		(layer "B.SilkS")
 		(effects
@@
 	)
 	(gr_text "JP3 capture rail"
-		(at 186 113.2 0)
-		(layer "B.SilkS")
-		(effects
-			(font
-				(size 0.8 0.8)
+		(at 188 113.6 0)
+		(layer "B.SilkS")
+		(effects
+			(font
+				(size 0.8 0.8)
+				(thickness 0.15)
+			)
+			(justify left mirror)
+		)
+	)
+	(gr_text "AFE Test Board v1   2026-10"
+		(at 136 119.2 0)
+		(layer "B.SilkS")
+		(effects
+			(font
+				(size 0.9 0.9)
 				(thickness 0.15)
 			)
@@
 	)
 	(gr_text "PMOD (J3)"
-		(at 198 109 0)
+		(at 204 109.4 0)
 		(layer "B.SilkS")
 		(effects
@@
 	)
 	(gr_text "1 CS    7 BIG_N"
-		(at 198 110.5 0)
+		(at 204 110.8 0)
 		(layer "B.SilkS")
 		(effects
@@
 	)
 	(gr_text "2 -     8 -"
-		(at 198 112 0)
+		(at 204 112.2 0)
 		(layer "B.SilkS")
 		(effects
@@
 	)
 	(gr_text "3 SDO   9 -"
-		(at 198 113.5 0)
+		(at 204 113.6 0)
 		(layer "B.SilkS")
 		(effects
@@
 	)
 	(gr_text "4 SCK  10 WAKE_N"
-		(at 198 115 0)
+		(at 204 115 0)
 		(layer "B.SilkS")
 		(effects
@@
 	)
 	(gr_text "5 GND  11 GND"
-		(at 198 116.5 0)
+		(at 204 116.4 0)
 		(layer "B.SilkS")
 		(effects
@@
 	)
 	(gr_text "6 3V3  12 3V3"
-		(at 198 118 0)
+		(at 204 117.8 0)
 		(layer "B.SilkS")
 		(effects
@@
 		)
 	)
-	(gr_text "AFE Test Board"
-		(at 158 116.5 0)
-		(layer "B.SilkS")
-		(effects
-			(font
-				(size 1.4 1.4)
-				(thickness 0.15)
-			)
+	(gr_text "Auselia"
+		(at 136 116.6 0)
+		(layer "B.SilkS")
+		(effects
+			(font
+				(size 1.7 1.7)
+				(thickness 0.15)
+			)

Commit message: Back silk: Oct 2026
Co-Authored-By: Claude Sonnet 5.5 <noreply@anthropic.com>
Other:
- board text added: "AFE Test Board v1 Oct 2026"
- board text removed: "AFE Test Board v1 2026-10"
Changed lines of the file:
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@@
 		)
 	)
-	(gr_text "AFE Test Board v1   2026-10"
+	(gr_text "AFE Test Board v1   Oct 2026"
 		(at 136 119.2 0)
 		(layer "B.SilkS")
